File: electronics/propulsion_control_module/electronic_speed_controller/electronic_speed_controller.kicad_sch (KiCad schematic)
At the start: 0 parts

Commit message: designing the propulsion controller ESC pt.5
Parts:
- added C1: 100nF, symbol Device:C
- added C2: 4.7uF, symbol Device:C
- added U1: STM32G071KBUxN, Package_DFN_QFN:QFN-32-1EP_5x5mm_P0.5mm_EP3.45x3.45mm, symbol MCU_ST_STM32G0:STM32G071KBUxN
Connections:
- new net GND: C1.2, C2.2, U1.33 (VSS), U1.5 (VSS)
- new net VDD_MCU: C1.1, C2.1, U1.4 (VDD)

Commit message: designing the propulsion controller ESC pt.6
Parts:
- added C10, C11, C9: 1uF, symbol Device:C
- added C3, C4, C5, C6, C7: 10uF, symbol Device:C
- added C8: 100uF, symbol Device:C
- added D1, D2, D3: 1N4148W, Diode_SMD:D_SOD-123, symbol Diode:1N4148W
- added J1: Power, symbol Connector_Generic:Conn_01x02
- added Q1, Q2, Q3, Q4, Q5, Q6: SiR696DP, Package_SO:PowerPAK_SO-8_Single, symbol Transistor_FET:SiR696DP
- added U2: HT7550-1-SOT89, Package_TO_SOT_SMD:SOT-89-3, symbol Regulator_Linear:HT75xx-1-SOT89
- added U3: HT7533-1-SOT89, Package_TO_SOT_SMD:SOT-89-3, symbol Regulator_Linear:HT75xx-1-SOT89
- added U4: DRV8300, VQFN-24-1EP_4x4mm_P0.5mm_EP2.45x2.45mm, symbol meridian:DRV8300
- added U5: TPS7A45xxKTT, Package_TO_SOT_SMD:TO-263-5_TabPin3, symbol Regulator_Linear:TPS7A45xxKTT
Connections:
- net GND: now also C3.2, C4.2, C5.2, C6.2, C7.2, C8.2, J1.2 (Pin_2), U2.1 (GND), U3.1 (GND), U4.6 (GND)
- new net: Q5.1 (S), Q5.2 (S), Q5.3 (S)
- new net: C10.1, D2.1 (K), U4.17 (BSTB)
- new net: Q3.1 (S), Q3.2 (S), Q3.3 (S)
- new net: Q1.1 (S), Q1.2 (S), Q1.3 (S)
- new net: Q4.1 (S), Q4.2 (S), Q4.3 (S)
- new net: C9.1, D1.1 (K), U4.20 (BSTA)
- new net: C11.1, D3.1 (K), U4.14 (BSTC)
- new net: Q6.1 (S), Q6.2 (S), Q6.3 (S)
- new net: Q2.1 (S), Q2.2 (S), Q2.3 (S)
- new net +3.3V: C6.1, U3.3 (VOUT)
- new net +5V: C4.1, C7.1, C8.1, D1.2 (A), D2.2 (A), D3.2 (A), U2.3 (VOUT), U4.4 (GVDD)
- new net +BATT: C3.1, C5.1, J1.1 (Pin_1), U2.2 (VIN), U3.2 (VIN)
- new net AHIGH: U4.22 (INHA)
- new net ALOW: U4.1 (INLA)
- new net BHIGH: U4.23 (INHB)
- new net BLOW: U4.2 (INLB)
- new net CHIGH: U4.24 (INHC)
- new net CLOW: U4.3 (INLC)
- new net GHA: U4.19 (GHA)
- new net GHB: U4.16 (GHB)
- new net GHC: U4.13 (GHC)
- new net GLA: U4.11 (GLA)
- new net GLB: U4.10 (GLB)
- new net GLC: U4.9 (GLC)
- new net MOTORA: C9.2, U4.18 (SHA)
- new net MOTORB: C10.2, U4.15 (SHB)
- new net MOTORC: C11.2, U4.12 (SHC)
- no-connect marks 0 -> 2

Commit message: designing the propulsion controller ESC pt.7
Parts:
- added C12, C13: 100uF, symbol Device:C
- added R1, R2, R3, R4, R5, R6: 20R, symbol Device:R
- added R10, R11, R12, R13, R14, R15, R16, R17, R9: 10R, symbol Device:R
- added R7: 1mR, symbol Device:R
- added R8: 1kR, symbol Device:R
- added U6: INA180B1, Package_TO_SOT_SMD:SOT-23-5, symbol Amplifier_Current:INA180B1
Connections:
- net +3.3V: now also C13.1, U6.5 (V+)
- net +BATT: now also Q1.5 (D), Q3.5 (D), Q5.5 (D)
- net GHA: now also R1.2
- net GHB: now also R3.2
- net GHC: now also R5.2
- net GLA: now also R2.2
- net GLB: now also R4.2
- net GLC: now also R6.2
- net GND: now also C12.2, C13.2, R10.1, R13.1, R16.1, R7.1, U6.2 (GND), U6.3 (-)
- net MOTORA: now also Q1.1 (S), Q1.2 (S), Q1.3 (S), Q2.5 (D), R14.1
- net MOTORB: now also Q3.1 (S), Q3.2 (S), Q3.3 (S), Q4.5 (D), R11.1
- net MOTORC: now also Q5.1 (S), Q5.2 (S), Q5.3 (S), Q6.5 (D), R17.1
- net at Q5.4 (G): now also R5.1
- net at Q3.4 (G): now also R3.1
- net at Q1.4 (G): now also R1.1
- net MOSFET_SOURCE: now reaches Q4.1 (S), Q4.2 (S), Q4.3 (S)
- net MOSFET_SOURCE: now also Q2.1 (S), Q2.2 (S), Q2.3 (S), Q6.1 (S), Q6.2 (S), Q6.3 (S), R7.2, U6.1 (+)
- net at Q4.4 (G): now also R4.1
- net at Q6.4 (G): now also R6.1
- net at Q2.4 (G): now also R2.1
- new net: R8.2, U6.4
- new net: R12.2, R15.2, R9.2
- new net BEMFA: R15.1, R16.2, R17.2
- new net BEMFB: R10.2, R11.2, R9.1
- new net BEMFC: R12.1, R13.2, R14.2
- new net CURRENT: C12.1, R8.1
Other:
- moved on the sheet: C1, C2, Q1, Q2, Q3, Q4, Q5, Q6, U1, U5

Commit message: forgot to commit ESC schematic changes
Parts:
- removed U5: TPS7A45xxKTT, Package_TO_SOT_SMD:TO-263-5_TabPin3, symbol Regulator_Linear:TPS7A45xxKTT
- R10, R13, R16: value 10R -> 1k
- R7: value 1mR -> 1m
Connections:
- net BEMF_COMMON: now reaches R12.2, R15.2, R9.2
Other:
- moved on the sheet: C1, C10, C11, C12, C13, C2, C3, C4, C5, C6, C7, C8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
