File: electronics/compute_module_carrier/M.2_E_and_M_Keys.kicad_sch (KiCad schematic)
At the start: 25 parts, among them J3 Bus_M.2_Socket_E, J4 Bus_M.2_Socket_M

Commit message: designing the compute module carrier pt.5
Connections:
- net ~{CLKREQM}: no longer J3.53 (~{CLKREQ0}), R20.1
- new net ~{CLKREQE}: J3.53 (~{CLKREQ0}), R20.1
Changed lines of the file:
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@@
 		)
 	)
-	(hierarchical_label "~{CLKREQM}"
+	(hierarchical_label "~{CLKREQE}"
 		(shape input)
 		(at 179.07 166.37 180)
