File: electronics/compute_module_carrier/LattePanda_Mu.kicad_sch (KiCad schematic)
At the start: 6 parts, among them J2 Conn_01x02_Pin

Commit message: designing the compute module carrier pt.4
Parts:
- removed J2: Conn_01x02_Pin, symbol Connector:Conn_01x02_Pin
- added H1, H2: MountingHole_Pad, symbol Mechanical:MountingHole_Pad
- added J2: Conn_01x03_Pin, symbol Connector:Conn_01x03_Pin
Connections:
- net GND: now also H1.1, H2.1, J2.3 (Pin_3)
- net at A1.10 (SIO_UART_TX): now also J2.1 (Pin_1)
- net at A1.12 (SIO_UART_RX): now also J2.2 (Pin_2)
- net ~{CLKREQ3}: now reaches A1.100 (~{CLKREQ3})
- net ~{CLKREQ4}: now reaches A1.102 (~{CLKREQ4})
- net ~{PEWAKE}: now reaches A1.103 (~{WAKE})
- net ~{PLT_RST}: now reaches A1.105 (~{PLTRST})
- net USB_2_P5-: now reaches A1.109 (USB2_P5-)
- net USB_2_P5+: now reaches A1.111 (USB2_P5+)
- net SUSCLK_WIFI: now reaches A1.131 (SUSCLK)
- net SOC_UART0_RX: now reaches A1.137 (UART0_RXD)
- net SOC_UART2_TX: now reaches A1.138 (UART2_TXD)
- net SOC_UART0_TX: now reaches A1.139 (UART0_TXD)
- net SOC_UART2_RX: now reaches A1.140 (UART2_RXD)
- net SOC_UART1_RX: now reaches A1.141 (UART1_RXD)
- net I2C5_SCL: now reaches A1.142 (I2C5_SCL)
- net SOC_UART1_TX: now reaches A1.143 (UART1_TXD)
- net I2C5_SDA: now reaches A1.144 (I2C5_SDA)
- net I2C4_SCL: now reaches A1.146 (I2C4_SCL)
- net I2C4_SDA: now reaches A1.148 (I2C4_SDA)
- net I2C3_SCL: now reaches A1.150 (I2C3_SCL)
- net I2C3_SDA: now reaches A1.152 (I2C3_SDA)
- net I2C2_SCL: now reaches A1.154 (I2C2_SCL)
- net I2C2_SDA: now reaches A1.156 (I2C2_SDA)
- net REFCLK0+: now reaches A1.85 (REFCLK0+)
- net REFCLK0-: now reaches A1.87 (REFCLK0-)
- net REFCLK3+: now reaches A1.88 (REFCLK3+)
- net REFCLK3-: now reaches A1.90 (REFCLK3-)
- net REFCLK4+: now reaches A1.94 (REFCLK4+)
- net REFCLK4-: now reaches A1.96 (REFCLK4-)
- net REFCLK2+: now reaches A1.97 (REFCLK2+)
- net REFCLK2-: now reaches A1.99 (REFCLK2-)
- no-connect marks 33 -> 89
Other:
- moved on the sheet: A1, BT1, R1, R14, R15

Commit message: designing the compute module carrier pt.6
Changed lines of the file:
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@@
 	)
 	(hierarchical_label "SOC_UART2_TX"
-		(shape input)
+		(shape output)
 		(at 335.28 208.28 0)
 		(effects
@@
 	)
 	(hierarchical_label "SOC_UART0_TX"
-		(shape input)
+		(shape output)
 		(at 335.28 198.12 0)
 		(effects
@@
 	)
 	(hierarchical_label "SOC_UART1_TX"
-		(shape input)
+		(shape output)
 		(at 335.28 203.2 0)
 		(effects
